Commit message: wrist_rot is end effector

File: code/robotarmudf/.ipynb_checkpoints/arm_urdf-checkpoint.urdf (robot description, URDF)
Before this commit: robot robot_arm, 6 links, 5 joints
Joints:
- joint elbow_joint: limit lower=-1.92 upper=1.92 -> lower=-1.61 upper=1.54
- joint shoulder_joint: limit lower=-1.57 upper=1.57 -> lower=-1.40 upper=1.75
- joint wrist_joint: limit lower=-1.57 upper=2.8 -> lower=-1.40 upper=1.75
- joint wrist_rot_joint: limit lower=-1.78 upper=0.48 -> lower=-1.57 upper=1.57
