Commit message: code
inverse kinematics code and arm urdf

File: code/robotarmudf/arm_urdf.urdf (robot description, URDF)
Before this commit: robot robot_arm, 6 links, 5 joints
Links:
- added link tool_tip
Joints:
- added joint tool_joint: type fixed, parent gripper, child tool_tip, origin xyz=0 0 0.155 rpy=0 0 0
- joint elbow_joint: axis 1 0 0 -> 0 1 0; limit lower=-1.61 upper=1.54 -> lower=-1.60 upper=1.53
- joint shoulder_joint: axis 1 0 0 -> 0 1 0; limit lower=-1.40 upper=1.75 -> lower=-1.57 upper=1.57
- joint wrist_joint: axis -1 0 0 -> 0 -1 0; limit lower=-1.40 upper=1.75 -> lower=-1.57 upper=2.8
- joint wrist_rot_joint: limit lower=-1.57 upper=1.57 -> lower=-1.78 upper=0.48

Commit message: update

File: code/robotarmudf/arm_urdf.urdf (robot description, URDF)
Before this commit: robot robot_arm, 7 links, 6 joints
Links:
- link arm1: geometry visual cylinder length=0.195 radius=0.022
- link base_rot: geometry visual cylinder length=0.066 radius=0.075
- link gripper: geometry visual box size=0.045 0.005 0.145
Joints:
- joint elbow_joint: origin xyz=0 0 0.2 rpy=0 0 0 -> xyz=0 0 0.195 rpy=0 0 0
- joint shoulder_joint: origin xyz=0 0 0.024 rpy=0 0 0 -> xyz=0 0 0.066 rpy=0 0 0
- joint tool_joint: origin xyz=0 0 0.155 rpy=0 0 0 -> xyz=0 0 0.145 rpy=0 0 0
- joint wrist_joint: limit lower=-1.57 upper=2.8 -> lower=-1.4 upper=1.75
